File: TMP76C75T.sch (KiCad schematic (older format))
At the start: 48 parts, among them J1 Conn_01x08_Male, J2 Conn_01x07_Male, J3 Conn_01x08_Male, J3-2 Conn_01x08_Male, J4 Conn_01x08_Male, J4-2 Conn_01x08_Male, J4-ADDR1 Conn_01x08_Male, J5 Conn_01x08_Male, J6 Conn_01x06_Male, J7 Conn_01x08_Male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

Commit message: Added via labels
Connections:
- net labels added: AN-, CE, OE
- wire segments 438 -> 437
Other:
- moved on the sheet: C13
Changed lines of the file:
@@
 U 1 1 61BDC390
 P 4600 4950
-F 0 "U1" H 5744 4946 50  0000 L CNN
-F 1 "TMP76C75T" H 5600 5750 50  0000 L CNN
+F 0 "U1" H 5744 4946 50  0000 C CNN
+F 1 "TMP76C75T" H 4600 4750 50  0000 C CNN
 F 2 "Package_LCC:PLCC-68_THT-Socket" H 4600 4950 50  0001 C CNN
 F 3 "" H 4600 4950 50  0001 C CNN
@@
 L Connector:Conn_01x08_Male J1
 U 1 1 62BEFC75
-P 1900 5400
-F 0 "J1" H 1872 5282 50  0000 R CNN
-F 1 "Conn_01x08_Male" H 1872 5373 50  0000 R CNN
-F 2 "Connector_PinSocket_2.54mm:PinSocket_1x08_P2.54mm_Vertical" H 1900 5400 50  0001 C CNN
-F 3 "~" H 1900 5400 50  0001 C CNN
-	1    1900 5400
-	1    0    0    1
+P 1900 5300
+F 0 "J1" H 2050 5700 50  0000 R CNN
+F 1 "Conn_01x08_Male" V 1850 5600 50  0000 R CNN
+F 2 "Connector_PinSocket_2.54mm:PinSocket_1x08_P2.54mm_Vertical" H 1900 5300 50  0001 C CNN
+F 3 "~" H 1900 5300 50  0001 C CNN
+	1    1900 5300
+	1    0    0    -1
 $EndComp
 $Comp
@@
 L Connector:Conn_01x08_Male J7
 U 1 1 62CD1C2A
-P 4850 7700
-F 0 "J7" V 5000 8100 50  0000 R CNN
-F 1 "Conn_01x08_Male" V 4800 8000 50  0000 R CNN
-F 2 "Connector_PinSocket_2.54mm:PinSocket_1x08_P2.54mm_Vertical" H 4850 7700 50  0001 C CNN
-F 3 "~" H 4850 7700 50  0001 C CNN
-	1    4850 7700
-	0    1    -1   0
+P 4750 7700
+F 0 "J7" V 4900 8150 50  0000 R CNN
+F 1 "Conn_01x08_Male" V 4700 8000 50  0000 R CNN
+F 2 "Connector_PinSocket_2.54mm:PinSocket_1x08_P2.54mm_Vertical" H 4750 7700 50  0001 C CNN
+F 3 "~" H 4750 7700 50  0001 C CNN
+	1    4750 7700
+	0    -1   -1   0
 $EndComp
 $Comp
@@
 U 1 1 6341A6B6
 P 3900 7700
-F 0 "J6" V 4050 7400 50  0000 R CNN
+F 0 "J6" V 4050 8050 50  0000 R CNN
 F 1 "Conn_01x06_Male" V 3850 8000 50  0000 R CNN
 F 2 "Connector_PinSocket_2.54mm:PinSocket_1x06_P2.54mm_Vertical" H 3900 7700 50  0001 C CNN
@@
 U 1 1 636AA39F
 P 3150 4500
-F 0 "J2" H 3100 4550 50  0000 C CNN
-F 1 "Conn_01x07_Male" H 2800 4450 50  0000 C CNN
+F 0 "J2" H 3250 4900 50  0000 C CNN
+F 1 "Conn_01x07_Male" V 3100 4500 50  0000 C CNN
 F 2 "Connector_PinSocket_2.54mm:PinSocket_1x07_P2.54mm_Vertical" H 3150 4500 50  0001 C CNN
 F 3 "~" H 3150 4500 50  0001 C CNN
@@
 	8200 3550 8200 4500
 Wire Wire Line
-	8200 4500 9200 4500
-Wire Wire Line
 	8250 3500 8250 4600
 Wire Wire Line
@@
 	4550 7500 4550 7350
 Wire Wire Line
-	4650 7500 4650 7350
+	4650 7500 4650 7400
 Wire Wire Line
 	4750 7500 4750 7350
@@
 Wire Wire Line
 	4950 7500 4950 7350
-Wire Wire Line
-	5050 7500 5050 7350
 Wire Wire Line
 	5150 7500 5150 7350
@@
 	2450 5700 2450 7200
 Connection ~ 5300 7200
-Wire Wire Line
-	5300 6200 5300 6300
 Wire Wire Line
 	6200 5300 6200 7200
@@
 L Device:C_Small C13
 U 1 1 66588547
-P 5400 6300
-F 0 "C13" V 5400 6100 50  0000 C CNN
-F 1 "C_Small" V 5400 6600 50  0000 C CNN
-F 2 "Capacitor_SMD:C_1206_3216Metric" H 5400 6300 50  0001 C CNN
-F 3 "~" H 5400 6300 50  0001 C CNN
-	1    5400 6300
+P 5400 6350
+F 0 "C13" V 5400 6150 50  0000 C CNN
+F 1 "C_Small" V 5400 6650 50  0000 C CNN
+F 2 "Capacitor_SMD:C_1206_3216Metric" H 5400 6350 50  0001 C CNN
+F 3 "~" H 5400 6350 50  0001 C CNN
+	1    5400 6350
 	0    1    1    0
 $EndComp
-Connection ~ 5300 6300
-Wire Wire Line
-	5300 6300 5300 7200
 Wire Wire Line
 	5200 6200 5200 6250
 Wire Wire Line
 	5200 6250 5500 6250
-Wire Wire Line
-	5500 6250 5500 6300
 $Comp
 L Device:C_Small C14
@@
 Text Notes 10750 7650 2    50   ~ 0
 v0.5
-Connection ~ 4150 3800
-Wire Wire Line
-	4200 3800 4150 3800
 $Comp
 L Connector:Conn_01x08_Male J4-ADDR1
@@
 P2.2
 Wire Wire Line
+	9200 4500 8200 4500
+Text Label 9000 4500 0    50   ~ 0
+CE
+Text Label 9000 4600 0    50   ~ 0
+OE
+Wire Wire Line
+	5300 6350 5300 7200
+Wire Wire Line
+	5300 6200 5300 6350
+Connection ~ 5300 6350
+Wire Wire Line
+	5500 6250 5500 6350
+Text Label 5500 6250 0    50   ~ 0
+AN-
+Wire Wire Line
+	5050 7350 5050 7500
+Wire Wire Line
 	7850 4100 9200 4100

Commit message: Fixes and nice updates
Fixed power rails for M303, fixed reset line tied to cap, added ground headers, adde clock header
Parts:
- added J-CLK2: Conn_01x02_Male, Connector_PinHeader_2.54mm:PinHeader_1x02_P2.54mm_Vertical, symbol Connector:Conn_01x02_Male
- added J-CNTL1: Conn_01x03_Male, Connector_PinHeader_2.54mm:PinHeader_1x03_P2.54mm_Vertical, symbol Connector:Conn_01x03_Male
- added J-GND1, J-GND2, J-GND3, J-GND4: Conn_01x02, Connector_PinHeader_2.54mm:PinHeader_1x02_P2.54mm_Vertical, symbol Connector_Generic:Conn_01x02
Connections:
- wire segments 437 -> 459
Other:
- moved on the sheet: C14, C15, C4, C5, C6
